File: Hardware/SMARTCONTROL2.brd (EAGLE design)
At the start: 40 x 54 mm, 36 parts, among them IC1 ESP12-SMT, J1 ESPFLASH-1X6-2.54-SOCKET, Q2 RJU003N03, Q3 RJU003N03, Q4 RJU003N03, Q5 RJU003N03

Commit message: Routing.
Parts:
- moved S1 38.2 mm to (4.50, 32.5)
- moved S2 21.6 mm to (4.50, 28.5), turned to 0 degrees
- moved R7 4.00 mm to (9.00, 21.0)
- moved R1 2.00 mm to (9.00, 19.0)
- moved R6 2.00 mm to (9.00, 17.0)
- moved C1 1.00 mm to (8.00, 47.0)
- moved C6 1.00 mm to (8.00, 37.0)
- moved REG1 1.00 mm to (9.00, 42.0)
- moved C8 0.50 mm to (9.00, 23.5), turned to 180 degrees
- moved R9 0.50 mm to (9.00, 11.0)
Routing:
- net !RESET: track 11.1 -> 66.1 mm
- net CH_PD: track 0.00 -> 31.2 mm, vias 0 -> 2
- net BUTTON1: track 11.0 -> 35.4 mm, vias 0 -> 2
- net 5V: track 86.0 -> 110.1 mm, vias 0 -> 4
- net GPIO12: track 0.00 -> 17.5 mm
- net GPIO0: track 23.4 -> 34.6 mm
- net BUTTON4: track 41.2 -> 49.7 mm, vias 0 -> 1
- net BUTTON2: track 31.8 -> 38.3 mm, vias 0 -> 1
- net GPIO15: track 8.98 -> 3.15 mm, vias 2 -> 0
- net BUTTON3: track 30.1 -> 34.7 mm, vias 0 -> 1
- net GND: track 7.99 -> 4.11 mm
- net N$27: track 0.02 -> 2.58 mm
- net 12V: track 43.1 -> 41.6 mm
- net 3.3V: track 27.1 -> 25.5 mm, vias 9 -> 10
- net ESP_RX: track 14.0 -> 14.9 mm
Other:
- board text added: "3V3"
- board text added: "ESPFlash"
- board text added: "ESP_RX"
- board text added: "ESP_TX"
- board text added: "IO0"
- board text added: "RST"
- board text removed: "3.3V"
- board text removed: "RX"
- board text removed: "TX"
